Commit message: update

File: src/rmitbot/urdf/rmitbot_imu.xacro (robot description, xacro)
@@ -1,5 +1,4 @@
 <?xml version="1.0"?>
 <robot xmlns:xacro="http://www.ros.org/wiki/xacro" name="rmitbot">
-  <!-- <xacro:macro name="imu_sensor" params="parent"> -->
     <link name="imu_link">
       <inertial>
@@ -85,4 +84,3 @@
     </sensor>
   </gazebo>
-  <!-- </xacro:macro> -->
 </robot>

File: src/rmitbot/urdf/rmitbot_platform.xacro (robot description, xacro)
@@ -1,3 +1,3 @@
-<?xml version="1.0" encoding="utf-8"?>
+<?xml version="1.0"?>
 <robot xmlns:xacro="http://www.ros.org/wiki/xacro" name="rmitbot">
   <link name="base_footprint"/>

File: src/rmitbot/urdf/rmitbot_ros2_control.xacro (robot description, xacro)
@@ -4,5 +4,6 @@
         <hardware>
             <plugin>gz_ros2_control/GazeboSimSystem</plugin>
-        </hardware> -->
+        </hardware>
+    -->
     <ros2_control name="RobotSystem" type="system">
         <hardware>
@@ -56,5 +57,5 @@
         </sensor>
     </ros2_control>
-    <gazebo>
+    <!-- <gazebo>
         <plugin filename="gz_ros2_control-system" name="gz_ros2_control::GazeboSimROS2ControlPlugin">
             <parameters>$(find rmitbot_controller)/config/rmitbot_controller.yaml</parameters>
@@ -63,4 +64,4 @@
             </ros>
         </plugin>
-    </gazebo>
+    </gazebo> -->
 </robot>
